File: 12.D1/pcb/ESP32_S3_Sensor_Shield/ESP32_S3_Sensor_Shield.kicad_pcb (KiCad board)
At the start: 2 copper layers, 85 x 69 mm, 8 parts, among them J1 ESP32_S3_L_H, J2 ESP32_S3_R_H, J3 MPU6050, J4 HCM5883L

Commit message: 12.D1更新PCB原理图与配套文档；12.D2完成全套传感器标定： 1. 清理self_raw多余嵌套空目录； 2. 生成3被试6类人体活动raw/calibrated两套数据集； 3. 产出calib_params.json、标定报告.md、标定前后对比图； 4. 新增数据集生成、绘图Python脚本； 5. 清理zip压缩包、KiCad临时锁定文件。
Parts:
- J4: value HCM5883L -> HMC5883L
Changed lines of the file:
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@@
 			)
 		)
-		(property "Value" "HCM5883L"
+		(property "Value" "HMC5883L"
 			(at 0 12.54 0)
 			(layer "F.Fab")
